Commit message: reduce hardware performance overhead

File: src/livox_laser_simulation/urdf/mid360.xacro (robot description, xacro)
@@ -3,5 +3,5 @@
   <xacro:property name="M_PI" value="3.1415926"/>
   <xacro:property name="laser_min_range" value="0.1"/>
-  <xacro:property name="laser_max_range" value="200.0"/>
+  <xacro:property name="laser_max_range" value="20.0"/>
   <xacro:property name="samples" value="30000"/>
   <xacro:property name="resolution" value="0.002"/>
@@ -67,5 +67,5 @@
           <visualize>false</visualize>
           <samples>${samples}</samples>
-          <downsample>1</downsample>
+          <downsample>3</downsample>
           <csv_file_name>$(find ros2_livox_simulation)/scan_mode/mid360.csv</csv_file_name>
           <topic>${topic}</topic>

Commit message: fix bug

File: src/livox_laser_simulation/urdf/mid360.xacro (robot description, xacro)
@@ -24,5 +24,5 @@
         <origin xyz="0.025 -0.0265 -0.025" rpy="${pi/2} 0 ${pi}"/>
         <geometry>
-          <mesh filename="model://mid360.stl" scale="0.0008 0.0008 0.0008"/>
+          <mesh filename="$(find ros2_livox_simulation)/meshes/mid360.stl" scale="0.0008 0.0008 0.0008"/>
         </geometry>
       </visual>

Commit message: add original config

File: src/livox_laser_simulation/urdf/mid360.xacro (robot description, xacro)
@@ -3,5 +3,5 @@
   <xacro:property name="M_PI" value="3.1415926"/>
   <xacro:property name="laser_min_range" value="0.1"/>
-  <xacro:property name="laser_max_range" value="20.0"/>
+  <xacro:property name="laser_max_range" value="100.0"/>
   <xacro:property name="samples" value="30000"/>
   <xacro:property name="resolution" value="0.002"/>
